Commit message: fixed joystick head control

File: sheldon_description/urdf/head.urdf.xacro (robot description, xacro)
@@ -9,5 +9,5 @@
    <xacro:property name="head_depth_camera_offset_y" value="0.000" />
    <xacro:property name="head_depth_camera_offset_z" value="0.025" /> <!-- 350 from bottom of torso? -->
-   <xacro:property name="head_depth_camera_rotation" value="0.0" /> <!-- rotation  -->
+   <xacro:property name="head_depth_camera_tilt" value="0.16" /> <!-- rotation  -->
   <xacro:macro name="head" params="name parent color *origin">
     <!-- Head Link -->
@@ -63,5 +63,5 @@
   <realsense_d435_camera name = "nuitrack_camera" parent = "head" color="Green">
      <origin xyz="${head_depth_camera_offset_x} ${head_depth_camera_offset_y} ${head_depth_camera_offset_z}"
-             rpy="0 ${head_depth_camera_rotation} 0" />
+             rpy="0 ${head_depth_camera_tilt} 0" />
   </realsense_d435_camera>
    <!-- Attach Astra camera in the head
