Commit message: modified URDF for gripping

File: sheldon_description/urdf/arm.urdf.xacro (robot description, xacro)
@@ -9,4 +9,11 @@
   <xacro:property name="lower_arm_size_y" value="0.065" />
   <xacro:property name="lower_arm_size_z" value="0.110" />
+  <xacro:property name="finger_size_x" value="0.020" />
+  <xacro:property name="finger_size_y" value="0.035" />
+  <xacro:property name="finger_size_z" value="0.120" />
+  <xacro:property name="finger_joint_offset_x" value="0.0" />
+  <xacro:property name="finger_joint_offset_y" value="0.035" />
+  <xacro:property name="finger_joint_offset_z" value="0.085" />
+  <xacro:property name="gripper_target_offset_z" value="0.180" />
   <xacro:property name="rx28_servo_width" value="0.035" />
   <xacro:property name="wrist_servo_offset_x" value="-0.008" /> <!--  -0.008 wrist center is slightly behind forearm center  -->
@@ -167,5 +174,5 @@
       <origin xyz="0 0 0.0235" rpy="0 0 0"/>
     </rx28_side_revolute>
-    <!-- Claw fixed link -->
+    <!-- Claw fixed joint -->
     <joint name="${side}_claw_fixed_joint" type="fixed">
       <origin xyz="0 0 0" rpy="0 0 0"/>
@@ -173,4 +180,5 @@
       <child link="${side}_claw_link" />
     </joint>
+    <!-- Claw body fixed link -->
     <link name="${side}_claw_link">
       <inertial>
@@ -196,4 +204,51 @@
       </collision>
     </link>
+    <!-- Finger Rotate -->
+    <joint name="${side}_finger_joint" type="revolute">
+      <axis xyz="1 0 0"/>
+      <limit effort="1000.0" lower="0.0" upper="0.548" velocity="0.5"/>
+      <origin rpy="-0.20 0 0" xyz="${finger_joint_offset_x} -${finger_joint_offset_y} ${finger_joint_offset_z}"/>
+      <parent link="${side}_claw_link"/>
+      <child link="${side}_finger_link1"/>
+    </joint>
+    <link name="${side}_finger_link1">
+      <visual>
+        <origin rpy="0.0 0.0 0.0" xyz="0 -0.008 ${finger_size_z/2}"/>
+        <geometry>
+          <box size="${finger_size_x} ${finger_size_y} ${finger_size_z}" />
+        </geometry>
+      </visual>
+    </link>
+    <joint name="${side}_finger_joint2" type="revolute">
+      <mimic joint="${side}_finger_joint" />
+      <axis xyz="-1 0 0"/>
+      <limit effort="1000.0" lower="0.0" upper="0.548" velocity="0.5"/>
+      <origin rpy="0.20 0 0" xyz="${finger_joint_offset_x} ${finger_joint_offset_y} ${finger_joint_offset_z}"/>
+      <parent link="${side}_claw_link"/>
+      <child link="${side}_finger_link2"/>
+    </joint>
+    <link name="${side}_finger_link2">
+      <visual>
+        <origin rpy="0.0 0.0 0.0" xyz="0 0.008 ${finger_size_z/2}"/>
+        <geometry>
+          <box size="${finger_size_x} ${finger_size_y} ${finger_size_z}" />
+        </geometry>
+      </visual>
+    </link>
+    <!-- Planning link and joint for the right gripper -->
+    <joint name="${side}_gripper_joint" type="fixed">
+      <origin rpy="${PI/2} 0 0" xyz="0 0 ${gripper_target_offset_z}"/>
+      <axis xyz="0 0 1" />
+      <parent link="${side}_claw_link"/>
+      <child link="${side}_gripper_link"/>
+    </joint>
+    <link name="${side}_gripper_link">
+      <visual>
+        <origin xyz="0 0 0" rpy="0 0 0"/>
+        <geometry>
+           <box size="0.001 0.0005 0.0005"/>
+        </geometry>
+      </visual>
+    </link>
   </xacro:macro>
 </robot>

Commit message: created first moveit config

File: sheldon_description/urdf/arm.urdf.xacro (robot description, xacro)
@@ -218,4 +218,5 @@
           <box size="${finger_size_x} ${finger_size_y} ${finger_size_z}" />
         </geometry>
+        <material name="Mustard"/>
       </visual>
     </link>
@@ -234,4 +235,5 @@
           <box size="${finger_size_x} ${finger_size_y} ${finger_size_z}" />
         </geometry>
+        <material name="Mustard"/>
       </visual>
     </link>
@@ -249,4 +251,5 @@
            <box size="0.001 0.0005 0.0005"/>
         </geometry>
+        <material name="Orange"/>
       </visual>
     </link>

File: sheldon_description/urdf/body.urdf.xacro (robot description, xacro)
@@ -6,5 +6,5 @@
   <xacro:property name="tibia_offset_z" value="${base_deck}" />  <!-- distance above ground -->
   <xacro:property name="tibia_size_x" value="0.0726" />
-  <xacro:property name="tibia_size_y" value="0.3556" />
+  <xacro:property name="tibia_size_y" value="0.340" />
   <xacro:property name="tibia_size_z" value="0.110" />
   <xacro:property name="knee_llimit" value="-0.175" />
@@ -15,5 +15,5 @@
   <xacro:property name="knee_offset_z" value="${tibia_size_z + 0.0}" /> <!-- knee sits on top of tibia -->
   <xacro:property name="femur_size_x" value="0.072" />
-  <xacro:property name="femur_size_y" value="0.356" />
+  <xacro:property name="femur_size_y" value="0.340" />
   <xacro:property name="femur_size_z" value="0.280" />
   <xacro:property name="waist_llimit" value="-0.175" />

File: sheldon_description/urdf/head.urdf.xacro (robot description, xacro)
@@ -6,7 +6,7 @@
   <xacro:property name="head_collision_offset_x" value="0.050" />
   <xacro:property name="head_collision_offset_y" value="0.020" />
-   <xacro:property name="head_depth_camera_offset_x" value="0.100" />
-   <xacro:property name="head_depth_camera_offset_y" value="0.0" />
-   <xacro:property name="head_depth_camera_offset_z" value="0.0" /> <!-- 350 from bottom of torso? -->
+   <xacro:property name="head_depth_camera_offset_x" value="0.050" />
+   <xacro:property name="head_depth_camera_offset_y" value="0.000" />
+   <xacro:property name="head_depth_camera_offset_z" value="0.025" /> <!-- 350 from bottom of torso? -->
    <xacro:property name="head_depth_camera_rotation" value="0.0" /> <!-- rotation  -->
   <xacro:macro name="head" params="name parent color *origin">

Commit message: MoveIt work in progress, changed claw to gripper

File: sheldon_description/urdf/arm.urdf.xacro (robot description, xacro)
@@ -174,12 +174,12 @@
       <origin xyz="0 0 0.0235" rpy="0 0 0"/>
     </rx28_side_revolute>
-    <!-- Claw fixed joint -->
-    <joint name="${side}_claw_fixed_joint" type="fixed">
+    <!-- Gripper fixed joint -->
+    <joint name="${side}_gripper_fixed_joint" type="fixed">
       <origin xyz="0 0 0" rpy="0 0 0"/>
       <parent link="${side}_wrist_rotate_link"/>
-      <child link="${side}_claw_link" />
-    </joint>
-    <!-- Claw body fixed link -->
-    <link name="${side}_claw_link">
+      <child link="${side}_gripper_body_link" />
+    </joint>
+    <!-- Gripper body fixed link -->
+    <link name="${side}_gripper_body_link">
       <inertial>
         <mass value="0.00001" />
@@ -205,12 +205,12 @@
     </link>
     <!-- Finger Rotate -->
-    <joint name="${side}_finger_joint" type="revolute">
+    <joint name="${side}_gripper_finger_joint" type="revolute">
       <axis xyz="1 0 0"/>
       <limit effort="1000.0" lower="0.0" upper="0.548" velocity="0.5"/>
       <origin rpy="-0.20 0 0" xyz="${finger_joint_offset_x} -${finger_joint_offset_y} ${finger_joint_offset_z}"/>
-      <parent link="${side}_claw_link"/>
-      <child link="${side}_finger_link1"/>
-    </joint>
-    <link name="${side}_finger_link1">
+      <parent link="${side}_gripper_body_link"/>
+      <child link="${side}_gripper_finger_link1"/>
+    </joint>
+    <link name="${side}_gripper_finger_link1">
       <visual>
         <origin rpy="0.0 0.0 0.0" xyz="0 -0.008 ${finger_size_z/2}"/>
@@ -221,13 +221,13 @@
       </visual>
     </link>
-    <joint name="${side}_finger_joint2" type="revolute">
-      <mimic joint="${side}_finger_joint" />
+    <joint name="${side}_gripper_finger_joint2" type="revolute">
+      <mimic joint="${side}_gripper_finger_joint" />
       <axis xyz="-1 0 0"/>
       <limit effort="1000.0" lower="0.0" upper="0.548" velocity="0.5"/>
       <origin rpy="0.20 0 0" xyz="${finger_joint_offset_x} ${finger_joint_offset_y} ${finger_joint_offset_z}"/>
-      <parent link="${side}_claw_link"/>
-      <child link="${side}_finger_link2"/>
-    </joint>
-    <link name="${side}_finger_link2">
+      <parent link="${side}_gripper_body_link"/>
+      <child link="${side}_gripper_finger_link2"/>
+    </joint>
+    <link name="${side}_gripper_finger_link2">
       <visual>
         <origin rpy="0.0 0.0 0.0" xyz="0 0.008 ${finger_size_z/2}"/>
@@ -238,9 +238,9 @@
       </visual>
     </link>
-    <!-- Planning link and joint for the right gripper -->
+    <!-- Planning link and joint for the gripper -->
     <joint name="${side}_gripper_joint" type="fixed">
       <origin rpy="${PI/2} 0 0" xyz="0 0 ${gripper_target_offset_z}"/>
       <axis xyz="0 0 1" />
-      <parent link="${side}_claw_link"/>
+      <parent link="${side}_gripper_body_link"/>
       <child link="${side}_gripper_link"/>
     </joint>

File: sheldon_description/urdf/sheldon.urdf (robot description, URDF)
Before this commit: robot sheldon_robot, 51 links, 50 joints
Links:
- removed link left_arm_claw_link
- removed link left_arm_finger_link1
- removed link left_arm_finger_link2
- removed link right_arm_claw_link
- removed link right_arm_finger_link1
- removed link right_arm_finger_link2
- added link left_arm_gripper_body_link, mass 0.00001; collision box size=0.05 0.12 0.215; visual mesh filename=package://sheldon_description/meshes/sheldon_claw.stl scale=0.1 0.1 0.1
- added link left_arm_gripper_finger_link1; visual box size=0.02 0.035 0.12
- added link left_arm_gripper_finger_link2; visual box size=0.02 0.035 0.12
- added link right_arm_gripper_body_link, mass 0.00001; collision box size=0.05 0.12 0.215; visual mesh filename=package://sheldon_description/meshes/sheldon_claw.stl scale=0.1 0.1 0.1
- added link right_arm_gripper_finger_link1; visual box size=0.02 0.035 0.12
- added link right_arm_gripper_finger_link2; visual box size=0.02 0.035 0.12
Joints:
- removed joint left_arm_claw_fixed_joint
- removed joint left_arm_finger_joint
- removed joint left_arm_finger_joint2
- removed joint right_arm_claw_fixed_joint
- removed joint right_arm_finger_joint
- removed joint right_arm_finger_joint2
- added joint left_arm_gripper_finger_joint: type revolute, parent left_arm_gripper_body_link, child left_arm_gripper_finger_link1, origin xyz=0.0 -0.035 0.085 rpy=-0.20 0 0, axis 1 0 0, limit lower=0.0 upper=0.548 effort=1000.0 velocity=0.5
- added joint left_arm_gripper_finger_joint2: type revolute, parent left_arm_gripper_body_link, child left_arm_gripper_finger_link2, origin xyz=0.0 0.035 0.085 rpy=0.20 0 0, axis -1 0 0, limit lower=0.0 upper=0.548 effort=1000.0 velocity=0.5, mimic joint=left_arm_gripper_finger_joint
- added joint left_arm_gripper_fixed_joint: type fixed, parent left_arm_wrist_rotate_link, child left_arm_gripper_body_link, origin xyz=0 0 0 rpy=0 0 0
- added joint right_arm_gripper_finger_joint: type revolute, parent right_arm_gripper_body_link, child right_arm_gripper_finger_link1, origin xyz=0.0 -0.035 0.085 rpy=-0.20 0 0, axis 1 0 0, limit lower=0.0 upper=0.548 effort=1000.0 velocity=0.5
- added joint right_arm_gripper_finger_joint2: type revolute, parent right_arm_gripper_body_link, child right_arm_gripper_finger_link2, origin xyz=0.0 0.035 0.085 rpy=0.20 0 0, axis -1 0 0, limit lower=0.0 upper=0.548 effort=1000.0 velocity=0.5, mimic joint=right_arm_gripper_finger_joint
- added joint right_arm_gripper_fixed_joint: type fixed, parent right_arm_wrist_rotate_link, child right_arm_gripper_body_link, origin xyz=0 0 0 rpy=0 0 0
- joint left_arm_gripper_joint: parent left_arm_claw_link -> left_arm_gripper_body_link
- joint right_arm_gripper_joint: parent right_arm_claw_link -> right_arm_gripper_body_link

Commit message: setting servo limits - WIP

File: sheldon_description/urdf/arm.urdf.xacro (robot description, xacro)
@@ -2,14 +2,13 @@
 <robot name="arm" xmlns:xacro="http://ros.org/wiki/xacro">
   <!-- Define a number of dimensions using properties -->
-  <!-- Define a number of dimensions using properties -->
   <xacro:property name="upper_arm_size_x" value="0.305" />
-  <xacro:property name="upper_arm_size_y" value="0.100" />
-  <xacro:property name="upper_arm_size_z" value="0.100" />
-  <xacro:property name="lower_arm_size_x" value="0.050" />
-  <xacro:property name="lower_arm_size_y" value="0.065" />
+  <xacro:property name="upper_arm_size_y" value="0.090" />
+  <xacro:property name="upper_arm_size_z" value="0.090" />
+  <xacro:property name="lower_arm_size_x" value="0.040" />
+  <xacro:property name="lower_arm_size_y" value="0.060" />
   <xacro:property name="lower_arm_size_z" value="0.110" />
   <xacro:property name="finger_size_x" value="0.020" />
   <xacro:property name="finger_size_y" value="0.035" />
-  <xacro:property name="finger_size_z" value="0.120" />
+  <xacro:property name="finger_size_z" value="0.110" />
   <xacro:property name="finger_joint_offset_x" value="0.0" />
   <xacro:property name="finger_joint_offset_y" value="0.035" />
@@ -18,8 +17,4 @@
   <xacro:property name="rx28_servo_width" value="0.035" />
   <xacro:property name="wrist_servo_offset_x" value="-0.008" /> <!--  -0.008 wrist center is slightly behind forearm center  -->
-<!--
-  <xacro:property name="knee_llimit" value="-0.175" />
-  <xacro:property name="knee_ulimit" value="0.873" />
-  <xacro:property name="knee_vlimit" value="1.571" />  velocity limit -->
   <xacro:property name="servo_bracket_color" value="Grey" />
   <xacro:macro name="arm" params="side reflect parent skin_color servo_color *origin">
@@ -39,5 +34,5 @@
       <!-- NOTE: right arm needs to be backwards to match servo feedback!
                  so we don't use reflect here! -->
-      <limit effort="30" velocity="0.524" lower="-3.14" upper="3.14" />
+      <limit effort="30" velocity="1.50" lower="-3.14" upper="3.14" />
       <parent link="${side}_shoulder_rotate_servo_link"/>
       <child link="${side}_shoulder_rotate_link" />
@@ -69,5 +64,5 @@
       <origin xyz="0.0869955 0 0" rpy="0 0 0"/>
       <axis xyz="0 1 0"/>
-      <limit effort="30" velocity="0.524" lower="-1.57" upper="2.617" />
+      <limit effort="30" velocity="1.50" lower="-0.6" upper="2.2" />
       <parent link="${side}_shoulder_rotate_link"/>
       <child link="${side}_shoulder_lift_servo_link" />
@@ -117,5 +112,5 @@
       </visual>
       <collision>
-        <origin xyz="${upper_arm_size_x/2} 0 0 " rpy="0 0 0" />
+        <origin xyz="${(upper_arm_size_x/2)+0.040} 0 0 " rpy="0 0 0" />
         <geometry>
           <box size="${upper_arm_size_x} ${upper_arm_size_y} ${upper_arm_size_z}" />
@@ -127,5 +122,5 @@
       <origin xyz="0.335 ${reflect * 0.015} 0" rpy="-1.57 ${1.57+(reflect * 1.57)} -1.57"/>      <!-- WIP!!! rpy="-1.57 0 -1.57" -->
     </dynamixel_rx64_pan>
-    <rx64_side_revolute parent="${side}_elbow_rotate_servo_link" name="${side}_elbow_rotate" llimit="-1.57" ulimit="1.57" vlimit="0.524" color="${servo_bracket_color}">
+    <rx64_side_revolute parent="${side}_elbow_rotate_servo_link" name="${side}_elbow_rotate" llimit="-2.50" ulimit="3.10" vlimit="3.0" color="${servo_bracket_color}">
       <origin xyz="0 0 0.0235" rpy="0 0 0"/>
     </rx64_side_revolute>
@@ -135,5 +130,5 @@
       <!-- <origin xyz="0 0 0" rpy="0 0 0"/> -->
     </dynamixel_rx64_tilt>
-    <rx64_hinge parent="${side}_elbow_bend_servo_link" name="${side}_elbow_bend" llimit="-1.57" ulimit="3.14" vlimit="0.785" color="${servo_bracket_color}">
+    <rx64_hinge parent="${side}_elbow_bend_servo_link" name="${side}_elbow_bend" llimit="-1.00" ulimit="3.0" vlimit="3.0" color="${servo_bracket_color}">
       <origin xyz="0 0 0.0" rpy="0 0 0"/>
     </rx64_hinge>
@@ -161,7 +156,7 @@
       </visual>
       <collision>
-        <origin xyz="0 0 ${lower_arm_size_z/2}" rpy="0 0 0" /> <!-- rpy="-1.57 0 0" -->
-        <geometry>
-          <box size="${lower_arm_size_x} ${lower_arm_size_y} ${lower_arm_size_z}" />
+        <origin xyz="0 0 ${lower_arm_size_z/2.0}" rpy="0 0 0" /> <!-- rpy="-1.57 0 0"   divide a little more then 1/2 for collision-->
+        <geometry>
+          <box size="${lower_arm_size_x} ${lower_arm_size_y} ${lower_arm_size_z * 0.90}" />
         </geometry>
       </collision>
@@ -171,5 +166,5 @@
       <origin xyz="${wrist_servo_offset_x} 0 ${lower_arm_size_z + (rx28_servo_width/2)}" rpy="0 0 3.14"/> <!-- <origin xyz="0 0 0.14" -->
     </dynamixel_rx28_pan>
-    <rx28_side_revolute parent="${side}_wrist_rotate_servo_link" name="${side}_wrist_rotate" llimit="-1.57" ulimit="1.57" vlimit="0.524" color="${servo_bracket_color}">
+    <rx28_side_revolute parent="${side}_wrist_rotate_servo_link" name="${side}_wrist_rotate" llimit="-2.9" ulimit="1.57" vlimit="3.0" color="${servo_bracket_color}">
       <origin xyz="0 0 0.0235" rpy="0 0 0"/>
     </rx28_side_revolute>
@@ -200,5 +195,5 @@
         <origin xyz="0 0 ${0.215 / 2.0}" rpy="0 0 0" /> <!-- rpy="-1.57 0 0" -->
         <geometry>
-          <box size="0.05 0.12 0.215"/>
+          <box size="0.05 0.09 0.180"/>
         </geometry>
       </collision>
@@ -207,5 +202,5 @@
     <joint name="${side}_gripper_finger_joint" type="revolute">
       <axis xyz="1 0 0"/>
-      <limit effort="1000.0" lower="0.0" upper="0.548" velocity="0.5"/>
+      <limit effort="1000.0" lower="0.0" upper="0.548" velocity="1.0"/>
       <origin rpy="-0.20 0 0" xyz="${finger_joint_offset_x} -${finger_joint_offset_y} ${finger_joint_offset_z}"/>
       <parent link="${side}_gripper_body_link"/>
@@ -224,5 +219,5 @@
       <mimic joint="${side}_gripper_finger_joint" />
       <axis xyz="-1 0 0"/>
-      <limit effort="1000.0" lower="0.0" upper="0.548" velocity="0.5"/>
+      <limit effort="30.0" lower="0.0" upper="3.0" velocity="0.5"/>
       <origin rpy="0.20 0 0" xyz="${finger_joint_offset_x} ${finger_joint_offset_y} ${finger_joint_offset_z}"/>
       <parent link="${side}_gripper_body_link"/>

File: sheldon_description/urdf/body.urdf.xacro (robot description, xacro)
@@ -6,5 +6,5 @@
   <xacro:property name="tibia_offset_z" value="${base_deck}" />  <!-- distance above ground -->
   <xacro:property name="tibia_size_x" value="0.0726" />
-  <xacro:property name="tibia_size_y" value="0.340" />
+  <xacro:property name="tibia_size_y" value="0.320" /> <!-- 3.40 collides with gripper -->
   <xacro:property name="tibia_size_z" value="0.110" />
   <xacro:property name="knee_llimit" value="-0.175" />

File: sheldon_description/urdf/sheldon.urdf (robot description, URDF)
Before this commit: robot sheldon_robot, 51 links, 50 joints
Links:
- link left_arm_gripper_body_link: geometry collision box size=0.05 0.09 0.180; visual mesh filename=package://sheldon_description/meshes/sheldon_claw.stl scale=0.1 0.1 0.1
- link left_arm_gripper_finger_link1: geometry visual box size=0.02 0.035 0.11
- link left_arm_gripper_finger_link2: geometry visual box size=0.02 0.035 0.11
- link left_arm_lower_link: geometry collision box size=0.04 0.06 0.099; visual box size=0.04 0.06 0.11
- link left_arm_upper_link: geometry collision box size=0.305 0.09 0.09; visual mesh filename=package://sheldon_description/meshes/sheldon_left_arm_upper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 scale=0.1 0.1 0.1
- link right_arm_gripper_body_link: geometry collision box size=0.05 0.09 0.180; visual mesh filename=package://sheldon_description/meshes/sheldon_claw.stl scale=0.1 0.1 0.1
- link right_arm_gripper_finger_link1: geometry visual box size=0.02 0.035 0.11
- link right_arm_gripper_finger_link2: geometry visual box size=0.02 0.035 0.11
- link right_arm_lower_link: geometry collision box size=0.04 0.06 0.099; visual box size=0.04 0.06 0.11
- link right_arm_upper_link: geometry collision box size=0.305 0.09 0.09; visual mesh filename=package://sheldon_description/meshes/sheldon_right_arm_uppe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 scale=0.1 0.1 0.1
- link tibia_link: geometry collision box size=0.0726 0.32 0.11; visual mesh filename=package://sheldon_description/meshes/sheldon_lower_legs.stl scale=0.1 0.1 0.1
