Commit message: change _command to _joint, reflect right,left arms

File: sheldon_description/urdf/arm.urdf.xacro (robot description, xacro)
@@ -31,7 +31,5 @@
     <joint name="${side}_shoulder_rotate_joint" type="revolute">
       <origin xyz="0 0 0" rpy="-1.57 0 1.57"/>
-      <axis xyz="-1 0 0"/>
-      <!-- NOTE: right arm needs to be backwards to match servo feedback!
-                 so we don't use reflect here! -->
+      <axis xyz="${reflect * -1} 0 0"/>
       <limit effort="30" velocity="1.50" lower="-3.14" upper="3.14" />
       <parent link="${side}_shoulder_rotate_servo_link"/>
@@ -64,5 +62,5 @@
       <origin xyz="0.0869955 0 0" rpy="0 0 0"/>
       <axis xyz="0 1 0"/>
-      <limit effort="30" velocity="1.50" lower="-0.6" upper="2.2" />
+      <limit effort="30" velocity="1.50" lower="-0.050" upper="2.10" />
       <parent link="${side}_shoulder_rotate_link"/>
       <child link="${side}_shoulder_lift_servo_link" />
@@ -120,7 +118,7 @@
     <!-- Elbow Rotate -->
     <dynamixel_rx64_pan parent="${side}_upper_link" name="${side}_elbow_rotate_servo" color="Blue">
-      <origin xyz="0.335 ${reflect * 0.015} 0" rpy="-1.57 ${1.57+(reflect * 1.57)} -1.57"/>      <!-- WIP!!! rpy="-1.57 0 -1.57" -->
+      <origin xyz="0.335 ${reflect * 0.015} 0" rpy="-1.57 ${1.57+(reflect * 1.57)} -1.57"/>
     </dynamixel_rx64_pan>
-    <rx64_side_revolute parent="${side}_elbow_rotate_servo_link" name="${side}_elbow_rotate" llimit="-2.50" ulimit="3.10" vlimit="3.0" color="${servo_bracket_color}">
+    <rx64_side_revolute parent="${side}_elbow_rotate_servo_link" name="${side}_elbow_rotate" llimit="-2.20" ulimit="3.14" vlimit="3.0" color="${servo_bracket_color}" reflect="${-reflect}">
       <origin xyz="0 0 0.0235" rpy="0 0 0"/>
     </rx64_side_revolute>
@@ -130,5 +128,5 @@
       <!-- <origin xyz="0 0 0" rpy="0 0 0"/> -->
     </dynamixel_rx64_tilt>
-    <rx64_hinge parent="${side}_elbow_bend_servo_link" name="${side}_elbow_bend" llimit="-1.00" ulimit="3.0" vlimit="3.0" color="${servo_bracket_color}">
+    <rx64_hinge parent="${side}_elbow_bend_servo_link" name="${side}_elbow_bend" llimit="-1.20" ulimit="3.14" vlimit="3.0" color="${servo_bracket_color}">
       <origin xyz="0 0 0.0" rpy="0 0 0"/>
     </rx64_hinge>
@@ -166,5 +164,5 @@
       <origin xyz="${wrist_servo_offset_x} 0 ${lower_arm_size_z + (rx28_servo_width/2)}" rpy="0 0 3.14"/> <!-- <origin xyz="0 0 0.14" -->
     </dynamixel_rx28_pan>
-    <rx28_side_revolute parent="${side}_wrist_rotate_servo_link" name="${side}_wrist_rotate" llimit="-2.9" ulimit="1.57" vlimit="3.0" color="${servo_bracket_color}">
+    <rx28_side_revolute parent="${side}_wrist_rotate_servo_link" name="${side}_wrist_rotate" llimit="-3.0" ulimit="1.57" vlimit="3.0" color="${servo_bracket_color}" reflect="${-reflect}">
       <origin xyz="0 0 0.0235" rpy="0 0 0"/>
     </rx28_side_revolute>
@@ -202,5 +200,5 @@
     <joint name="${side}_gripper_finger_joint" type="revolute">
       <axis xyz="1 0 0"/>
-      <limit effort="1000.0" lower="0.0" upper="0.548" velocity="1.0"/>
+      <limit effort="30.0" lower="-0.10" upper="3.14" velocity="1.0"/>
       <origin rpy="-0.20 0 0" xyz="${finger_joint_offset_x} -${finger_joint_offset_y} ${finger_joint_offset_z}"/>
       <parent link="${side}_gripper_body_link"/>
@@ -219,5 +217,5 @@
       <mimic joint="${side}_gripper_finger_joint" />
       <axis xyz="-1 0 0"/>
-      <limit effort="30.0" lower="0.0" upper="3.0" velocity="0.5"/>
+      <limit effort="30.0" lower="-0.10" upper="3.14" velocity="0.5"/>
       <origin rpy="0.20 0 0" xyz="${finger_joint_offset_x} ${finger_joint_offset_y} ${finger_joint_offset_z}"/>
       <parent link="${side}_gripper_body_link"/>

File: sheldon_description/urdf/hardware/rx28.xacro (robot description, xacro)
@@ -59,8 +59,8 @@
     </link>
   </xacro:macro>
-  <xacro:macro name="rx28_side_revolute" params="parent name color llimit ulimit vlimit *origin">
+  <xacro:macro name="rx28_side_revolute" params="parent name color llimit ulimit vlimit *origin reflect=1">
     <joint name="${name}_joint" type="revolute">
       <xacro:insert_block name="origin" />
-       <axis xyz="0 0 1"/>
+       <axis xyz="0 0 ${reflect}"/>
       <limit effort="30" velocity="${vlimit}" lower="${llimit}" upper="${ulimit}" />
       <parent link="${parent}"/>

File: sheldon_description/urdf/hardware/rx64.xacro (robot description, xacro)
@@ -59,8 +59,8 @@
     </link>
   </xacro:macro>
-  <xacro:macro name="rx64_side_revolute" params="parent name color llimit ulimit vlimit *origin">
+  <xacro:macro name="rx64_side_revolute" params="parent name color llimit ulimit vlimit *origin reflect=1" >
     <joint name="${name}_joint" type="revolute">
       <xacro:insert_block name="origin" />
-       <axis xyz="0 0 1"/>
+       <axis xyz="0 0 ${reflect}"/>
       <limit effort="30" velocity="${vlimit}" lower="${llimit}" upper="${ulimit}" />
       <parent link="${parent}"/>

Commit message: moveit works on robot, motions are slow

File: sheldon_description/urdf/arm.urdf.xacro (robot description, xacro)
@@ -32,5 +32,5 @@
       <origin xyz="0 0 0" rpy="-1.57 0 1.57"/>
       <axis xyz="${reflect * -1} 0 0"/>
-      <limit effort="30" velocity="1.50" lower="-3.14" upper="3.14" />
+      <limit effort="90" velocity="2.50" lower="-3.14" upper="3.14" />
       <parent link="${side}_shoulder_rotate_servo_link"/>
       <child link="${side}_shoulder_rotate_link" />
@@ -62,5 +62,5 @@
       <origin xyz="0.0869955 0 0" rpy="0 0 0"/>
       <axis xyz="0 1 0"/>
-      <limit effort="30" velocity="1.50" lower="-0.050" upper="2.10" />
+      <limit effort="90" velocity="1.50" lower="-0.050" upper="2.10" />
       <parent link="${side}_shoulder_rotate_link"/>
       <child link="${side}_shoulder_lift_servo_link" />
@@ -200,5 +200,5 @@
     <joint name="${side}_gripper_finger_joint" type="revolute">
       <axis xyz="1 0 0"/>
-      <limit effort="30.0" lower="-0.10" upper="3.14" velocity="1.0"/>
+      <limit effort="90" lower="-0.10" upper="3.14" velocity="1.0"/>
       <origin rpy="-0.20 0 0" xyz="${finger_joint_offset_x} -${finger_joint_offset_y} ${finger_joint_offset_z}"/>
       <parent link="${side}_gripper_body_link"/>
@@ -217,5 +217,5 @@
       <mimic joint="${side}_gripper_finger_joint" />
       <axis xyz="-1 0 0"/>
-      <limit effort="30.0" lower="-0.10" upper="3.14" velocity="0.5"/>
+      <limit effort="90" lower="-0.10" upper="3.14" velocity="0.5"/>
       <origin rpy="0.20 0 0" xyz="${finger_joint_offset_x} ${finger_joint_offset_y} ${finger_joint_offset_z}"/>
       <parent link="${side}_gripper_body_link"/>

File: sheldon_description/urdf/sheldon.urdf (robot description, URDF)
Before this commit: robot sheldon_robot, 51 links, 50 joints
Joints:
- joint left_arm_elbow_bend_joint: limit lower=-1.57 upper=3.14 effort=30 velocity=0.785 -> lower=-1.2 upper=3.14 effort=30 velocity=3.0
- joint left_arm_elbow_rotate_joint: axis 0 0 1 -> 0 0 -1; limit lower=-1.57 upper=1.57 effort=30 velocity=0.524 -> lower=-2.2 upper=3.14 effort=30 velocity=3.0
- joint left_arm_gripper_finger_joint: limit lower=0.0 upper=0.548 effort=1000.0 velocity=0.5 -> lower=-0.10 upper=3.14 effort=30.0 velocity=1.0
- joint left_arm_gripper_finger_joint2: limit lower=0.0 upper=0.548 effort=1000.0 velocity=0.5 -> lower=-0.10 upper=3.14 effort=30.0 velocity=0.5
- joint left_arm_shoulder_lift_joint: limit lower=-1.57 upper=2.617 effort=30 velocity=0.524 -> lower=-0.050 upper=2.10 effort=30 velocity=1.50
- joint left_arm_shoulder_rotate_joint: limit lower=-3.14 upper=3.14 effort=30 velocity=0.524 -> lower=-3.14 upper=3.14 effort=30 velocity=1.50
- joint left_arm_wrist_rotate_joint: axis 0 0 1 -> 0 0 -1; limit lower=-1.57 upper=1.57 effort=30 velocity=0.524 -> lower=-3.0 upper=1.57 effort=30 velocity=3.0
- joint right_arm_elbow_bend_joint: limit lower=-1.57 upper=3.14 effort=30 velocity=0.785 -> lower=-1.2 upper=3.14 effort=30 velocity=3.0
- joint right_arm_elbow_rotate_joint: limit lower=-1.57 upper=1.57 effort=30 velocity=0.524 -> lower=-2.2 upper=3.14 effort=30 velocity=3.0
- joint right_arm_gripper_finger_joint: limit lower=0.0 upper=0.548 effort=1000.0 velocity=0.5 -> lower=-0.10 upper=3.14 effort=30.0 velocity=1.0
- joint right_arm_gripper_finger_joint2: limit lower=0.0 upper=0.548 effort=1000.0 velocity=0.5 -> lower=-0.10 upper=3.14 effort=30.0 velocity=0.5
- joint right_arm_shoulder_lift_joint: limit lower=-1.57 upper=2.617 effort=30 velocity=0.524 -> lower=-0.050 upper=2.10 effort=30 velocity=1.50
- joint right_arm_shoulder_rotate_joint: axis -1 0 0 -> 1 0 0; limit lower=-3.14 upper=3.14 effort=30 velocity=0.524 -> lower=-3.14 upper=3.14 effort=30 velocity=1.50
- joint right_arm_wrist_rotate_joint: limit lower=-1.57 upper=1.57 effort=30 velocity=0.524 -> lower=-3.0 upper=1.57 effort=30 velocity=3.0

Commit message: added forked dynamixel_motor, changes to support moveit

File: sheldon_description/urdf/arm.urdf.xacro (robot description, xacro)
@@ -7,5 +7,6 @@
   <xacro:property name="lower_arm_size_x" value="0.040" />
   <xacro:property name="lower_arm_size_y" value="0.060" />
-  <xacro:property name="lower_arm_size_z" value="0.110" />
+  <!-- <xacro:property name="lower_arm_size_z" value="0.110" /> -->  <!-- CORRECT VALUE!! -->
+  <xacro:property name="lower_arm_size_z" value="0.080" />  <!-- KLUDGE FOR TESTING!!! -->
   <xacro:property name="finger_size_x" value="0.020" />
   <xacro:property name="finger_size_y" value="0.035" />
@@ -32,5 +33,5 @@
       <origin xyz="0 0 0" rpy="-1.57 0 1.57"/>
       <axis xyz="${reflect * -1} 0 0"/>
-      <limit effort="90" velocity="2.50" lower="-3.14" upper="3.14" />
+      <limit effort="1000" velocity="2.3" lower="-3.14" upper="3.14" />
       <parent link="${side}_shoulder_rotate_servo_link"/>
       <child link="${side}_shoulder_rotate_link" />
@@ -62,5 +63,5 @@
       <origin xyz="0.0869955 0 0" rpy="0 0 0"/>
       <axis xyz="0 1 0"/>
-      <limit effort="90" velocity="1.50" lower="-0.050" upper="2.10" />
+      <limit effort="1000" velocity="4.6" lower="-0.050" upper="2.10" />
       <parent link="${side}_shoulder_rotate_link"/>
       <child link="${side}_shoulder_lift_servo_link" />
@@ -120,5 +121,5 @@
       <origin xyz="0.335 ${reflect * 0.015} 0" rpy="-1.57 ${1.57+(reflect * 1.57)} -1.57"/>
     </dynamixel_rx64_pan>
-    <rx64_side_revolute parent="${side}_elbow_rotate_servo_link" name="${side}_elbow_rotate" llimit="-2.20" ulimit="3.14" vlimit="3.0" color="${servo_bracket_color}" reflect="${-reflect}">
+    <rx64_side_revolute parent="${side}_elbow_rotate_servo_link" name="${side}_elbow_rotate" llimit="-2.20" ulimit="3.14" vlimit="6.6" color="${servo_bracket_color}" reflect="${-reflect}">
       <origin xyz="0 0 0.0235" rpy="0 0 0"/>
     </rx64_side_revolute>
@@ -128,10 +129,11 @@
       <!-- <origin xyz="0 0 0" rpy="0 0 0"/> -->
     </dynamixel_rx64_tilt>
-    <rx64_hinge parent="${side}_elbow_bend_servo_link" name="${side}_elbow_bend" llimit="-1.20" ulimit="3.14" vlimit="3.0" color="${servo_bracket_color}">
+    <rx64_hinge parent="${side}_elbow_bend_servo_link" name="${side}_elbow_bend" llimit="-1.20" ulimit="3.14" vlimit="6.6" color="${servo_bracket_color}">
       <origin xyz="0 0 0.0" rpy="0 0 0"/>
     </rx64_hinge>
     <!-- Lower Arm fixed link -->
     <joint name="${side}_lower_fixed_joint" type="fixed">
-      <origin xyz="0.030 0 0.031" rpy="0 1.57 0"/> <!-- .034... "0.14 0 0.05" half the length, plus bracket lenth and offset -->
+      <!--  "0.030 0 0.031" half the length, plus bracket lenth and offset -->
+      <origin xyz="0.030 0 0.031" rpy="0 1.57 0"/>  <!-- KLUDGE FOR TESTING!!! -->
       <parent link="${side}_elbow_bend_link"/>
       <child link="${side}_lower_link" />
@@ -160,14 +162,21 @@
       </collision>
     </link>
+    <!-- Wrist Bend (NEW!) -->
+    <dynamixel_rx28_tilt parent="${side}_lower_link" name="${side}_wrist_bend_servo" color="${servo_color}">
+      <origin xyz="0 0 ${lower_arm_size_z + (rx28_servo_width/2)}" rpy="0 -1.57 0"/>
+    </dynamixel_rx28_tilt>
+    <rx28_hinge parent="${side}_wrist_bend_servo_link" name="${side}_wrist_bend" llimit="-1.57" ulimit="1.57" vlimit="6.6" color="${servo_bracket_color}">
+      <origin xyz="0 0 0.0" rpy="0 0 0"/>
+    </rx28_hinge>
     <!-- Wrist Rotate -->
-    <dynamixel_rx28_pan parent="${side}_lower_link" name="${side}_wrist_rotate_servo" color="${servo_color}">
-      <origin xyz="${wrist_servo_offset_x} 0 ${lower_arm_size_z + (rx28_servo_width/2)}" rpy="0 0 3.14"/> <!-- <origin xyz="0 0 0.14" -->
+    <dynamixel_rx28_pan parent="${side}_wrist_bend_link" name="${side}_wrist_rotate_servo" color="${servo_color}">
+      <origin xyz="${(rx28_servo_width/2)+0.03} 0 0" rpy="3.14 -1.57 0" />
     </dynamixel_rx28_pan>
-    <rx28_side_revolute parent="${side}_wrist_rotate_servo_link" name="${side}_wrist_rotate" llimit="-3.0" ulimit="1.57" vlimit="3.0" color="${servo_bracket_color}" reflect="${-reflect}">
-      <origin xyz="0 0 0.0235" rpy="0 0 0"/>
+    <rx28_side_revolute parent="${side}_wrist_rotate_servo_link" name="${side}_wrist_rotate" llimit="-3.0" ulimit="1.57" vlimit="5.8" color="${servo_bracket_color}" reflect="${-reflect}">
+      <origin xyz="0 0 0" rpy="0 0 0"/>
     </rx28_side_revolute>
     <!-- Gripper fixed joint -->
     <joint name="${side}_gripper_fixed_joint" type="fixed">
-      <origin xyz="0 0 0" rpy="0 0 0"/>
+      <origin xyz="0 0 0" rpy="0 0 0"/>    <!-- "0 0.03 0" -->
       <parent link="${side}_wrist_rotate_link"/>
       <child link="${side}_gripper_body_link" />
@@ -193,5 +202,5 @@
         <origin xyz="0 0 ${0.215 / 2.0}" rpy="0 0 0" /> <!-- rpy="-1.57 0 0" -->
         <geometry>
-          <box size="0.05 0.09 0.180"/>
+          <box size="0.05 0.09 0.170"/>
         </geometry>
       </collision>
@@ -200,5 +209,5 @@
     <joint name="${side}_gripper_finger_joint" type="revolute">
       <axis xyz="1 0 0"/>
-      <limit effort="90" lower="-0.10" upper="3.14" velocity="1.0"/>
+      <limit effort="1000" lower="-0.10" upper="3.14" velocity="5.8"/>
       <origin rpy="-0.20 0 0" xyz="${finger_joint_offset_x} -${finger_joint_offset_y} ${finger_joint_offset_z}"/>
       <parent link="${side}_gripper_body_link"/>
@@ -217,5 +226,5 @@
       <mimic joint="${side}_gripper_finger_joint" />
       <axis xyz="-1 0 0"/>
-      <limit effort="90" lower="-0.10" upper="3.14" velocity="0.5"/>
+      <limit effort="1000" lower="-0.10" upper="3.14" velocity="5.8"/>
       <origin rpy="0.20 0 0" xyz="${finger_joint_offset_x} ${finger_joint_offset_y} ${finger_joint_offset_z}"/>
       <parent link="${side}_gripper_body_link"/>
@@ -233,5 +242,5 @@
     <!-- Planning link and joint for the gripper -->
     <joint name="${side}_gripper_joint" type="fixed">
-      <origin rpy="${PI/2} 0 0" xyz="0 0 ${gripper_target_offset_z}"/>
+      <origin rpy="0 ${PI/2} 0" xyz="0 0 ${gripper_target_offset_z}"/>
       <axis xyz="0 0 1" />
       <parent link="${side}_gripper_body_link"/>

File: sheldon_description/urdf/hardware/rx28.xacro (robot description, xacro)
@@ -63,5 +63,5 @@
       <xacro:insert_block name="origin" />
        <axis xyz="0 0 ${reflect}"/>
-      <limit effort="30" velocity="${vlimit}" lower="${llimit}" upper="${ulimit}" />
+      <limit effort="1000" velocity="${vlimit}" lower="${llimit}" upper="${ulimit}" />
       <parent link="${parent}"/>
       <child link="${name}_link" />
@@ -123,5 +123,5 @@
       <xacro:insert_block name="origin" />
        <axis xyz="0 1 0"/>
-      <limit effort="30" velocity="${vlimit}" lower="${llimit}" upper="${ulimit}" />
+      <limit effort="1000" velocity="${vlimit}" lower="${llimit}" upper="${ulimit}" />
       <parent link="${parent}"/>
       <child link="${name}_link" />

File: sheldon_description/urdf/hardware/rx64.xacro (robot description, xacro)
@@ -63,5 +63,5 @@
       <xacro:insert_block name="origin" />
        <axis xyz="0 0 ${reflect}"/>
-      <limit effort="30" velocity="${vlimit}" lower="${llimit}" upper="${ulimit}" />
+      <limit effort="1000" velocity="${vlimit}" lower="${llimit}" upper="${ulimit}" />
       <parent link="${parent}"/>
       <child link="${name}_link" />
@@ -94,5 +94,5 @@
       <xacro:insert_block name="origin" />
        <axis xyz="0 1 0"/>
-      <limit effort="30" velocity="${vlimit}" lower="${llimit}" upper="${ulimit}" />
+      <limit effort="1000" velocity="${vlimit}" lower="${llimit}" upper="${ulimit}" />
       <parent link="${parent}"/>
       <child link="${name}_link" />

File: sheldon_description/urdf/sheldon.urdf (robot description, URDF)
Before this commit: robot sheldon_robot, 51 links, 50 joints
Links:
- added link left_arm_wrist_bend_link, mass 0.00001; collision box size=0.030 0.045 0.031; visual mesh filename=package://sheldon_description/meshes/rx28-hinge-bracket.stl scale=1 1 1
- added link left_arm_wrist_bend_servo_link, mass 0.00001; collision box size=0.0506 0.045 0.0356; visual mesh filename=package://sheldon_description/meshes/rx28.stl scale=1 1 1
- added link right_arm_wrist_bend_link, mass 0.00001; collision box size=0.030 0.045 0.031; visual mesh filename=package://sheldon_description/meshes/rx28-hinge-bracket.stl scale=1 1 1
- added link right_arm_wrist_bend_servo_link, mass 0.00001; collision box size=0.0506 0.045 0.0356; visual mesh filename=package://sheldon_description/meshes/rx28.stl scale=1 1 1
- link left_arm_gripper_body_link: geometry collision box size=0.05 0.09 0.170; visual mesh filename=package://sheldon_description/meshes/sheldon_claw.stl scale=0.1 0.1 0.1
- link left_arm_lower_link: geometry collision box size=0.04 0.06 0.072; visual box size=0.04 0.06 0.08
- link right_arm_gripper_body_link: geometry collision box size=0.05 0.09 0.170; visual mesh filename=package://sheldon_description/meshes/sheldon_claw.stl scale=0.1 0.1 0.1
- link right_arm_lower_link: geometry collision box size=0.04 0.06 0.072; visual box size=0.04 0.06 0.08
Joints:
- added joint left_arm_wrist_bend_joint: type revolute, parent left_arm_wrist_bend_servo_link, child left_arm_wrist_bend_link, origin xyz=0 0 0.0 rpy=0 0 0, axis 0 1 0, limit lower=-1.57 upper=1.57 effort=1000 velocity=6.6
- added joint left_arm_wrist_bend_servo_joint: type fixed, parent left_arm_lower_link, child left_arm_wrist_bend_servo_link, origin xyz=0 0 0.0975 rpy=0 -1.57 0
- added joint right_arm_wrist_bend_joint: type revolute, parent right_arm_wrist_bend_servo_link, child right_arm_wrist_bend_link, origin xyz=0 0 0.0 rpy=0 0 0, axis 0 1 0, limit lower=-1.57 upper=1.57 effort=1000 velocity=6.6
- added joint right_arm_wrist_bend_servo_joint: type fixed, parent right_arm_lower_link, child right_arm_wrist_bend_servo_link, origin xyz=0 0 0.0975 rpy=0 -1.57 0
- joint head_pan_joint: limit lower=-1.57 upper=1.57 effort=30 velocity=0.524 -> lower=-1.57 upper=1.57 effort=1000 velocity=0.524
- joint head_sidetilt_joint: limit lower=-0.35 upper=0.35 effort=30 velocity=0.524 -> lower=-0.35 upper=0.35 effort=1000 velocity=0.524
- joint head_tilt_joint: limit lower=-0.6 upper=1.2 effort=30 velocity=0.524 -> lower=-0.6 upper=1.2 effort=1000 velocity=0.524
- joint left_arm_elbow_bend_joint: limit lower=-1.2 upper=3.14 effort=30 velocity=3.0 -> lower=-1.2 upper=3.14 effort=1000 velocity=6.6
- joint left_arm_elbow_rotate_joint: limit lower=-2.2 upper=3.14 effort=30 velocity=3.0 -> lower=-2.2 upper=3.14 effort=1000 velocity=6.6
- joint left_arm_gripper_finger_joint: limit lower=-0.10 upper=3.14 effort=30.0 velocity=1.0 -> lower=-0.10 upper=3.14 effort=1000 velocity=5.8
- joint left_arm_gripper_finger_joint2: limit lower=-0.10 upper=3.14 effort=30.0 velocity=0.5 -> lower=-0.10 upper=3.14 effort=1000 velocity=5.8
- joint left_arm_gripper_joint: origin xyz=0 0 0.18 rpy=1.570795 0 0 -> xyz=0 0 0.18 rpy=0 1.570795 0
- joint left_arm_shoulder_lift_joint: limit lower=-0.050 upper=2.10 effort=30 velocity=1.50 -> lower=-0.050 upper=2.10 effort=1000 velocity=4.6
- joint left_arm_shoulder_rotate_joint: limit lower=-3.14 upper=3.14 effort=30 velocity=1.50 -> lower=-3.14 upper=3.14 effort=1000 velocity=2.3
- joint left_arm_wrist_rotate_joint: limit lower=-3.0 upper=1.57 effort=30 velocity=3.0 -> lower=-3.0 upper=1.57 effort=1000 velocity=5.8; origin xyz=0 0 0.0235 rpy=0 0 0 -> xyz=0 0 0 rpy=0 0 0
- joint left_arm_wrist_rotate_servo_joint: origin xyz=-0.008 0 0.1275 rpy=0 0 3.14 -> xyz=0.0475 0 0 rpy=3.14 -1.57 0; parent left_arm_lower_link -> left_arm_wrist_bend_link
- joint right_arm_elbow_bend_joint: limit lower=-1.2 upper=3.14 effort=30 velocity=3.0 -> lower=-1.2 upper=3.14 effort=1000 velocity=6.6
- joint right_arm_elbow_rotate_joint: limit lower=-2.2 upper=3.14 effort=30 velocity=3.0 -> lower=-2.2 upper=3.14 effort=1000 velocity=6.6
- joint right_arm_gripper_finger_joint: limit lower=-0.10 upper=3.14 effort=30.0 velocity=1.0 -> lower=-0.10 upper=3.14 effort=1000 velocity=5.8
- joint right_arm_gripper_finger_joint2: limit lower=-0.10 upper=3.14 effort=30.0 velocity=0.5 -> lower=-0.10 upper=3.14 effort=1000 velocity=5.8
- joint right_arm_gripper_joint: origin xyz=0 0 0.18 rpy=1.570795 0 0 -> xyz=0 0 0.18 rpy=0 1.570795 0
- joint right_arm_shoulder_lift_joint: limit lower=-0.050 upper=2.10 effort=30 velocity=1.50 -> lower=-0.050 upper=2.10 effort=1000 velocity=4.6
- joint right_arm_shoulder_rotate_joint: limit lower=-3.14 upper=3.14 effort=30 velocity=1.50 -> lower=-3.14 upper=3.14 effort=1000 velocity=2.3
- joint right_arm_wrist_rotate_joint: limit lower=-3.0 upper=1.57 effort=30 velocity=3.0 -> lower=-3.0 upper=1.57 effort=1000 velocity=5.8; origin xyz=0 0 0.0235 rpy=0 0 0 -> xyz=0 0 0 rpy=0 0 0
- joint right_arm_wrist_rotate_servo_joint: origin xyz=-0.008 0 0.1275 rpy=0 0 3.14 -> xyz=0.0475 0 0 rpy=3.14 -1.57 0; parent right_arm_lower_link -> right_arm_wrist_bend_link
