Commit message: working on moveit options or alternatives

File: sheldon_description/urdf/arm.urdf.xacro (robot description, xacro)
@@ -10,6 +10,6 @@
   <xacro:property name="lower_arm_size_z" value="0.080" />  <!-- KLUDGE FOR TESTING!!! -->
   <xacro:property name="finger_size_x" value="0.020" />
-  <xacro:property name="finger_size_y" value="0.035" />
-  <xacro:property name="finger_size_z" value="0.110" />
+  <xacro:property name="finger_size_y" value="0.020" />
+  <xacro:property name="finger_size_z" value="0.080" />
   <xacro:property name="finger_joint_offset_x" value="0.0" />
   <xacro:property name="finger_joint_offset_y" value="0.035" />
@@ -216,5 +216,5 @@
     <link name="${side}_gripper_finger_link1">
       <visual>
-        <origin rpy="0.0 0.0 0.0" xyz="0 -0.008 ${finger_size_z/2}"/>
+        <origin rpy="0.0 0.0 0.0" xyz="0 -0.020 ${0.04+finger_size_z/2}"/>
         <geometry>
           <box size="${finger_size_x} ${finger_size_y} ${finger_size_z}" />
@@ -222,4 +222,10 @@
         <material name="Mustard"/>
       </visual>
+      <collision>
+        <origin rpy="0.0 0.0 0.0" xyz="0 -0.020 ${0.04+finger_size_z/2}"/>
+        <geometry>
+          <box size="${finger_size_x} ${finger_size_y} ${finger_size_z}" />
+        </geometry>
+      </collision>
     </link>
     <joint name="${side}_gripper_finger_joint2" type="revolute">
@@ -233,5 +239,5 @@
     <link name="${side}_gripper_finger_link2">
       <visual>
-        <origin rpy="0.0 0.0 0.0" xyz="0 0.008 ${finger_size_z/2}"/>
+        <origin rpy="0.0 0.0 0.0" xyz="0 0.020 ${0.04+finger_size_z/2}"/>
         <geometry>
           <box size="${finger_size_x} ${finger_size_y} ${finger_size_z}" />
@@ -239,4 +245,10 @@
         <material name="Mustard"/>
       </visual>
+      <collision>
+        <origin rpy="0.0 0.0 0.0" xyz="0 0.020 ${0.04+finger_size_z/2}"/>
+        <geometry>
+          <box size="${finger_size_x} ${finger_size_y} ${finger_size_z}" />
+        </geometry>
+      </collision>
     </link>
     <!-- Planning link and joint for the gripper -->

File: sheldon_description/urdf/base.urdf.xacro (robot description, xacro)
@@ -8,13 +8,13 @@
        All component positions are calculated relative to base_link  -->
   <!-- simplified box collision geometry for base -->
-  <xacro:property name="base_size_x" value="0.520" /> <!-- ~20"base length -->
+  <xacro:property name="base_size_x" value="0.550" /> <!-- ~22"base length -->
   <xacro:property name="base_size_y" value="0.3556" /> <!-- 14" base width -->
   <xacro:property name="base_size_z" value="0.094" />  <!-- base only, no ankle bone  "0.1524"-->
   <xacro:property name="base_ground_clearance" value="0.076" />
   <xacro:property name="base_deck" value="0.170" /> <!-- distance from ground to top of base -->
-  <xacro:property name="wheels_offset_x" value="0.0254" /> <!-- "0.0254" wheels 1" back from center -->
+  <xacro:property name="wheel_offset_x" value="-0.190" /> <!-- wheels distance back from center -->
   <xacro:property name="wheel_offset_y" value="0.2032" /> <!-- 1/2 base + center of wheel -->
-  <xacro:property name="wheel_length" value="0.0508" /> <!-- wheel width -->
-  <xacro:property name="wheel_radius" value="0.0762" />
+  <xacro:property name="wheel_width" value="0.0508"    /> <!-- wheel width -->
+  <xacro:property name="wheel_radius" value="0.0762"   />
   <!-- location of laser -->
   <xacro:property name="base_laser_x" value="0.150" />
@@ -28,5 +28,5 @@
       <limit effort="100" velocity="100"/>
       <safety_controller k_velocity="10" />
-      <origin xyz="0 ${reflect*wheel_offset_y} ${wheel_radius}" rpy="${reflect*1.57} 0 0" />
+      <origin xyz="${wheel_offset_x} ${reflect*wheel_offset_y} ${wheel_radius}" rpy="${reflect*1.57} 0 0" />
       <parent link="${parent}_link"/>
       <child link="${parent}_${suffix}_wheel_link"/>
@@ -36,8 +36,14 @@
         <origin xyz="0 0 0" rpy="0 0 0" />
         <geometry>
-          <cylinder radius="${wheel_radius}" length="${wheel_length}"/>
+          <cylinder radius="${wheel_radius}" length="${wheel_width}"/>
         </geometry>
         <material name="${color}" />
       </visual>
+      <collision>
+        <origin xyz="0 0 0" rpy="0 0 0" />
+        <geometry>
+          <box size="${wheel_radius*2.5} ${wheel_radius*2.5} ${wheel_width}" /> <!-- padding for wheel covers -->
+        </geometry>
+      </collision>
     </link>
   </xacro:macro>
@@ -47,5 +53,5 @@
     <link name="${name}_link">
       <visual>
-        <origin xyz="0 0 ${base_ground_clearance}" rpy="0 0 0" />
+        <origin xyz="-0.025 0 ${base_ground_clearance}" rpy="0 0 0" />
         <geometry>
           <mesh filename="package://sheldon_description/meshes/sheldon_base.stl" scale="0.1 0.1 0.1"/>
@@ -54,5 +60,5 @@
       </visual>
       <collision>
-        <origin xyz="${wheels_offset_x} 0 ${(base_ground_clearance + base_size_z) / 2}" rpy="0 0 0" />
+        <origin xyz="0 0 ${(base_ground_clearance + base_size_z) / 2}" rpy="0 0 0" />
         <geometry>
           <box size="${base_size_x} ${base_size_y} ${base_ground_clearance + base_size_z}" />
@@ -67,5 +73,5 @@
     <link name="base_footprint">
       <visual>
-        <origin xyz="${wheels_offset_x} 0 0" rpy="0 0 0" />
+        <origin xyz="0 0 0" rpy="0 0 0" />
         <geometry>
           <box size="${base_size_x} ${base_size_y} 0.001" />

File: sheldon_description/urdf/head.urdf.xacro (robot description, xacro)
@@ -54,5 +54,5 @@
       </visual>
       <collision>
-        <origin xyz="${head_collision_offset_x} ${-head_collision_offset_y} 0" rpy="0 0 -0.15" />
+        <origin xyz="${head_collision_offset_x} ${-head_collision_offset_y} 0" rpy="0 0 0" />
         <geometry>
           <box size="${head_size_x} ${head_size_y} ${head_size_z}" />

File: sheldon_description/urdf/sheldon.urdf (robot description, URDF)
Before this commit: robot sheldon_robot, 55 links, 54 joints
Links:
- link base_footprint: geometry visual box size=0.55 0.3556 0.001
- link base_l_wheel_link: geometry collision box size=0.1905 0.1905 0.0508; visual cylinder length=0.0508 radius=0.0762
- link base_link: geometry collision box size=0.55 0.3556 0.17; visual mesh filename=package://sheldon_description/meshes/sheldon_base.stl scale=0.1 0.1 0.1
- link base_r_wheel_link: geometry collision box size=0.1905 0.1905 0.0508; visual cylinder length=0.0508 radius=0.0762
- link left_arm_gripper_finger_link1: geometry collision box size=0.02 0.02 0.08; visual box size=0.02 0.02 0.08
- link left_arm_gripper_finger_link2: geometry collision box size=0.02 0.02 0.08; visual box size=0.02 0.02 0.08
- link right_arm_gripper_finger_link1: geometry collision box size=0.02 0.02 0.08; visual box size=0.02 0.02 0.08
- link right_arm_gripper_finger_link2: geometry collision box size=0.02 0.02 0.08; visual box size=0.02 0.02 0.08
Joints:
- joint base_l_wheel_joint: origin xyz=0 0.2032 0.0762 rpy=1.57 0 0 -> xyz=-0.19 0.2032 0.0762 rpy=1.57 0 0
- joint base_r_wheel_joint: origin xyz=0 -0.2032 0.0762 rpy=-1.57 0 0 -> xyz=-0.19 -0.2032 0.0762 rpy=-1.57 0 0
- joint nuitrack_camera_joint: origin xyz=0.05 0.0 0.025 rpy=0 0.0 0 -> xyz=0.05 0.0 0.025 rpy=0 0.16 0

Commit message: calibrated URDF values for accurate arm placement

File: sheldon_description/urdf/arm.urdf.xacro (robot description, xacro)
@@ -8,5 +8,5 @@
   <xacro:property name="lower_arm_size_y" value="0.060" />
   <!-- <xacro:property name="lower_arm_size_z" value="0.110" /> -->  <!-- CORRECT VALUE!! -->
-  <xacro:property name="lower_arm_size_z" value="0.080" />  <!-- KLUDGE FOR TESTING!!! -->
+  <xacro:property name="lower_arm_size_z" value="0.153" />  <!-- KLUDGE FOR TESTING!!! -->
   <xacro:property name="finger_size_x" value="0.020" />
   <xacro:property name="finger_size_y" value="0.020" />
@@ -15,5 +15,5 @@
   <xacro:property name="finger_joint_offset_y" value="0.035" />
   <xacro:property name="finger_joint_offset_z" value="0.085" />
-  <xacro:property name="gripper_target_offset_z" value="0.180" />
+  <xacro:property name="gripper_target_offset_z" value="0.210" />
   <xacro:property name="rx28_servo_width" value="0.035" />
   <xacro:property name="wrist_servo_offset_x" value="-0.008" /> <!--  -0.008 wrist center is slightly behind forearm center  -->

File: sheldon_description/urdf/base.urdf.xacro (robot description, xacro)
@@ -8,9 +8,8 @@
        All component positions are calculated relative to base_link  -->
   <!-- simplified box collision geometry for base -->
-  <xacro:property name="base_size_x" value="0.550" /> <!-- ~22"base length -->
-  <xacro:property name="base_size_y" value="0.3556" /> <!-- 14" base width -->
-  <xacro:property name="base_size_z" value="0.094" />  <!-- base only, no ankle bone  "0.1524"-->
-  <xacro:property name="base_ground_clearance" value="0.076" />
-  <xacro:property name="base_deck" value="0.170" /> <!-- distance from ground to top of base -->
+  <xacro:property name="base_size_x" value="0.559" /> <!-- 22"base length -->
+  <xacro:property name="base_size_y" value="0.366" /> <!-- base main body width .183mm x 2-->
+  <xacro:property name="base_ground_clearance" value="0.088" />
+  <xacro:property name="base_deck_top" value="0.185" /> <!-- distance from ground to top of base -->
   <xacro:property name="wheel_offset_x" value="-0.190" /> <!-- wheels distance back from center -->
   <xacro:property name="wheel_offset_y" value="0.2032" /> <!-- 1/2 base + center of wheel -->
@@ -19,5 +18,5 @@
   <!-- location of laser -->
   <xacro:property name="base_laser_x" value="0.150" />
-  <xacro:property name="base_laser_z" value="${base_deck + 0.0}" />
+  <xacro:property name="base_laser_z" value="${base_deck_top + 0.0}" />
   <xacro:property name="laser_height" value="0.040" />
   <xacro:property name="laser_radius" value="0.039" />
@@ -60,7 +59,7 @@
       </visual>
       <collision>
-        <origin xyz="0 0 ${(base_ground_clearance + base_size_z) / 2}" rpy="0 0 0" />
+        <origin xyz="0 0 ${(base_deck_top) / 2}" rpy="0 0 0" />
         <geometry>
-          <box size="${base_size_x} ${base_size_y} ${base_ground_clearance + base_size_z}" />
+          <box size="${base_size_x} ${base_size_y} ${base_deck_top}" />
         </geometry>
       </collision>

File: sheldon_description/urdf/body.urdf.xacro (robot description, xacro)
@@ -4,8 +4,8 @@
   <xacro:property name="tibia_offset_x" value="0.0" />
   <xacro:property name="tibia_offset_y" value="0.0" />
-  <xacro:property name="tibia_offset_z" value="${base_deck}" />  <!-- distance above ground -->
+  <xacro:property name="tibia_offset_z" value="${base_deck_top}" />  <!-- distance above ground -->
   <xacro:property name="tibia_size_x" value="0.0726" />
-  <xacro:property name="tibia_size_y" value="0.320" /> <!-- 3.40 collides with gripper -->
-  <xacro:property name="tibia_size_z" value="0.110" />
+  <xacro:property name="tibia_size_y" value="0.322" /> <!-- to outside edges of bearing tubes -->
+  <xacro:property name="tibia_size_z" value="0.109" /> <!-- .294 (measured height) - base_deck_top -->
   <xacro:property name="knee_llimit" value="-0.175" />
   <xacro:property name="knee_ulimit" value="0.873" />
@@ -16,5 +16,5 @@
   <xacro:property name="femur_size_x" value="0.072" />
   <xacro:property name="femur_size_y" value="0.340" />
-  <xacro:property name="femur_size_z" value="0.280" />
+  <xacro:property name="femur_size_z" value="0.281" /> <!-- .575 (measured height) - .294 (tibia height) -->
   <xacro:property name="hip_llimit" value="-0.175" />
   <xacro:property name="hip_ulimit" value="1.92" />

File: sheldon_description/urdf/robot.urdf.xacro (robot description, xacro)
@@ -7,6 +7,6 @@
    <xacro:property name="head_offset_z" value="0.440" />
    <xacro:property name="arm_offset_x" value="0.0" />
-   <xacro:property name="arm_offset_y" value="-0.146" />  <!-- from center of torso -->
-   <xacro:property name="arm_offset_z" value="0.385" />   <!-- from bottom of torso -->
+   <xacro:property name="arm_offset_y" value="-0.164" />  <!-- from center of torso -->
+   <xacro:property name="arm_offset_z" value="0.389" />   <!-- from bottom of torso -->
    <xacro:property name="front_astra_camera_offset_x" value="0.100" />
    <xacro:property name="front_astra_camera_offset_y" value="0.000" />

File: sheldon_description/urdf/sheldon.urdf (robot description, URDF)
Before this commit: robot sheldon_robot, 55 links, 54 joints
Links:
- link base_footprint: geometry visual box size=0.559 0.366 0.001
- link base_link: geometry collision box size=0.559 0.366 0.185; visual mesh filename=package://sheldon_description/meshes/sheldon_base.stl scale=0.1 0.1 0.1
- link femur_link: geometry collision box size=0.072 0.34 0.281; visual mesh filename=package://sheldon_description/meshes/sheldon_upper_legs.stl scale=0.1 0.1 0.1
- link left_arm_lower_link: geometry collision box size=0.04 0.06 0.1377; visual box size=0.04 0.06 0.153
- link right_arm_lower_link: geometry collision box size=0.04 0.06 0.1377; visual box size=0.04 0.06 0.153
- link tibia_link: geometry collision box size=0.0726 0.322 0.109; visual mesh filename=package://sheldon_description/meshes/sheldon_lower_legs.stl scale=0.1 0.1 0.1
Joints:
- joint base_body_joint: origin xyz=0.0 0.0 0.17 rpy=0 0 0 -> xyz=0.0 0.0 0.185 rpy=0 0 0
- joint hip_joint: origin xyz=0 0  0.28 rpy=0 0 0 -> xyz=0 0  0.281 rpy=0 0 0
- joint knee_joint: origin xyz=0 0  0.11 rpy=0 0 0 -> xyz=0 0  0.109 rpy=0 0 0
- joint left_arm_gripper_joint: origin xyz=0 0 0.18 rpy=0 1.570795 0 -> xyz=0 0 0.21 rpy=0 1.570795 0
- joint left_arm_torso_joint: origin xyz=0.0 0.146 0.385 rpy=0 0 0 -> xyz=0.0 0.164 0.389 rpy=0 0 0
- joint left_arm_wrist_bend_servo_joint: origin xyz=0 0 0.0975 rpy=0 -1.57 0 -> xyz=0 0 0.1705 rpy=0 -1.57 0
- joint lidar_base_joint: origin xyz=0.15 0 0.17 rpy=0 0 0 -> xyz=0.15 0 0.185 rpy=0 0 0
- joint right_arm_gripper_joint: origin xyz=0 0 0.18 rpy=0 1.570795 0 -> xyz=0 0 0.21 rpy=0 1.570795 0
- joint right_arm_torso_joint: origin xyz=0.0 -0.146 0.385 rpy=0 0 0 -> xyz=0.0 -0.164 0.389 rpy=0 0 0
- joint right_arm_wrist_bend_servo_joint: origin xyz=0 0 0.0975 rpy=0 -1.57 0 -> xyz=0 0 0.1705 rpy=0 -1.57 0
