Commit message: improved floor object accuracy

File: sheldon_description/urdf/base.urdf.xacro (robot description, xacro)
@@ -3,5 +3,5 @@
 <!--  <xacro:include filename="$(find sheldon_description)/urdf/sensors/hokuyo_urg_laser.urdf.xacro" />
 -->
-  <xacro:include filename="$(find sheldon_description)/urdf/_lplidar.urdf.xacro"/>
+  <xacro:include filename="$(find sheldon_description)/urdf/sensors/_lplidar.urdf.xacro"/>
   <!-- Sheldon Base definition.
        base_link is centered between wheels, at ground level.
@@ -18,5 +18,5 @@
   <!-- location of laser -->
   <xacro:property name="base_laser_x" value="0.150" />
-  <xacro:property name="base_laser_z" value="${base_deck_top + 0.0}" />
+  <xacro:property name="base_laser_z" value="${base_deck_top - 0.008}" />
   <xacro:property name="laser_height" value="0.040" />
   <xacro:property name="laser_radius" value="0.039" />
@@ -84,23 +84,5 @@
     <child link="base_link" />
   </joint>
-    <!-- Base mounted laser -->
-    <!-- Base to laser link
-    <joint name="base_laser_joint" type="fixed">
-      <origin xyz="${base_laser_x} 0 ${base_laser_z}" rpy="0 0 0" />
-      <parent link="base_link"/>
-      <child link="laser_link"/>
-    </joint>
-    -->
-    <!-- Laser definition
-    <link name="laser_link">
-      <visual>
-        <origin xyz="0 0 ${laser_height/2}" rpy="0 0 0" />
-        <geometry>
-          <cylinder length="${laser_height}" radius="${laser_radius}"/>
-        </geometry>
-        <material name="Red" />
-      </visual>
-    </link>
-    -->
+   <!-- Base mounted laser -->
    <sensor_lplidar parent = "base_link">
       <origin xyz="${base_laser_x} 0 ${base_laser_z}" rpy="0 0 0" />

File: sheldon_description/urdf/body.urdf.xacro (robot description, xacro)
@@ -26,10 +26,10 @@
   <xacro:property name="torso_size_y" value="0.355" />
   <xacro:property name="torso_size_z" value="0.457" />  <!--  to top of shoulder .5112 .7112 28 inch torso for now -->
-   <xacro:property name="chest_camera_servo_offset_x" value="0.090" />
+   <xacro:property name="chest_camera_servo_offset_x" value="0.110" /> <!--0.090 -->
    <xacro:property name="chest_camera_servo_offset_y" value="-0.098" />
-   <xacro:property name="chest_camera_servo_offset_z" value="0.380" /> <!-- 350 from bottom of torso? -->
-   <xacro:property name="chest_camera_offset_x" value="-0.044" />
-   <xacro:property name="chest_camera_offset_y" value="0.0" />
-   <xacro:property name="chest_camera_offset_z" value="0.08" />
+   <xacro:property name="chest_camera_servo_offset_z" value="0.350" /> <!-- 360 - from bottom of torso? -->
+   <xacro:property name="chest_camera_offset_x" value="0.00" /> <!-- 0.0  -->
+   <xacro:property name="chest_camera_offset_y" value="0.01" />  <!-- -0.02    global x -->
+   <xacro:property name="chest_camera_offset_z" value="0.128" />  <!-- 0.128   global y -->
    <xacro:property name="chest_camera_rotation" value="0.0" />
   <xacro:macro name="body" params="parent name color">
@@ -113,5 +113,5 @@
   <astra_camera name = "astra_camera" parent = "chest_camera_tilt" color="Green">
      <origin xyz="${chest_camera_offset_x} ${chest_camera_offset_y} ${chest_camera_offset_z}"
-     rpy="1.57 0 1.57" />
+     rpy="1.57 0.0 1.60" /> <!-- "1.57 0.0 1.57"  -->
   </astra_camera>
   </xacro:macro>

File: sheldon_description/urdf/head.urdf.xacro (robot description, xacro)
@@ -61,8 +61,8 @@
     </link>
    <!-- Attach d435 camera -->
-  <realsense_d435_camera name = "nuitrack_camera" parent = "head" color="Green">
+  <sensor_d435 name = "head_camera" parent = "head_link">
      <origin xyz="${head_depth_camera_offset_x} ${head_depth_camera_offset_y} ${head_depth_camera_offset_z}"
              rpy="0 ${head_depth_camera_tilt} 0" />
-  </realsense_d435_camera>
+  </sensor_d435>
    <!-- Attach Astra camera in the head
   <astra_camera name = "astra_camera2" parent = "head" color="Green">

File: sheldon_description/urdf/robot.urdf.xacro (robot description, xacro)
@@ -26,4 +26,7 @@
    <xacro:include filename="$(find sheldon_description)/urdf/hardware/ax12.xacro" />
    <xacro:include filename="$(find sheldon_description)/urdf/sensors/xtion_camera.xacro" />
+   <xacro:include filename="$(find sheldon_description)/urdf/sensors/_d435.urdf.xacro" />
+   <xacro:include filename="$(find sheldon_description)/urdf/sensors/_zr300.urdf.xacro"/>
+   <xacro:include filename="$(find sheldon_description)/urdf/sensors/astra_camera.urdf.xacro" />
    <xacro:include filename="$(find sheldon_description)/urdf/materials.urdf.xacro" />
    <xacro:include filename="$(find sheldon_description)/urdf/base.urdf.xacro" />
@@ -31,8 +34,8 @@
    <xacro:include filename="$(find sheldon_description)/urdf/head.urdf.xacro" />
    <xacro:include filename="$(find sheldon_description)/urdf/arm.urdf.xacro" />
-   <xacro:include filename="$(find sheldon_description)/urdf/astra_camera.urdf.xacro" />
+    <!--
    <xacro:include filename="$(find sheldon_description)/urdf/realsense_d435_camera.urdf.xacro" />
-   <xacro:include filename="$(find sheldon_description)/urdf/_zr300.urdf.xacro"/>
    <xacro:include filename="$(find sheldon_description)/urdf/depth_camera.urdf.xacro" />
+    -->
    <!-- Add the base and wheels -->
    <sheldon_base name="base" color="White"/>

File: sheldon_description/urdf/sensors/_d435.urdf.xacro (robot description, xacro)
@@ -7,5 +7,5 @@
 -->
 <robot name="sensor_d435" xmlns:xacro="http://ros.org/wiki/xacro">
-  <xacro:macro name="sensor_d435" params="parent *origin">
+  <xacro:macro name="sensor_d435" params="name parent *origin">
     <xacro:property name="M_PI" value="3.1415926535897931" />
     <!-- The following values are approximate, and the camera node

File: sheldon_description/urdf/sensors/astra_camera.urdf.xacro (robot description, xacro)
@@ -9,8 +9,8 @@
     <link name="${name}_link">
       <visual>
-        <origin xyz="0.03 0.02 0.085" rpy="1.57 0 1.57" />  <!-- rpy="0 0 -1.57"-->
+        <origin xyz="0.0 -0.04 0.00" rpy="1.57 0 1.57" />  <!-- 0.03 0.02 0.085  rpy="0 0 -1.57"-->
         <geometry>
           <!-- </mesh filename="package://tb2s_description/meshes/xtion.stl" scale="0.001 0.001 0.001"/> -->
-          <mesh filename="package://sheldon_description/meshes/astra.stl" scale="0.001 0.001 0.001"/>
+          <box size="0.08 0.02 0.02"/>
         </geometry>
         <material name="${color}" />
