Commit message: arduino publishes accurate /joint_state message values for knee and hip

File: sheldon_description/urdf/body.urdf.xacro (robot description, xacro)
@@ -17,10 +17,10 @@
   <xacro:property name="femur_size_y" value="0.340" />
   <xacro:property name="femur_size_z" value="0.280" />
-  <xacro:property name="waist_llimit" value="-0.175" />
-  <xacro:property name="waist_ulimit" value="1.92" />
-  <xacro:property name="waist_vlimit" value="1.571" /> <!-- velocity limit -->
-  <xacro:property name="waist_offset_x" value="0.0" />
-  <xacro:property name="waist_offset_y" value="0.0" />
-  <xacro:property name="waist_offset_z" value="${femur_size_z + 0.0}" /> <!-- waist sits on top of femur -->
+  <xacro:property name="hip_llimit" value="-0.175" />
+  <xacro:property name="hip_ulimit" value="1.92" />
+  <xacro:property name="hip_vlimit" value="1.571" /> <!-- velocity limit -->
+  <xacro:property name="hip_offset_x" value="0.0" />
+  <xacro:property name="hip_offset_y" value="0.0" />
+  <xacro:property name="hip_offset_z" value="${femur_size_z + 0.0}" /> <!-- hip sits on top of femur -->
   <xacro:property name="torso_size_x" value="0.230" />
   <xacro:property name="torso_size_y" value="0.355" />
@@ -72,8 +72,8 @@
       </collision>
     </link>
-    <joint name="waist_joint" type="revolute">
-      <origin xyz="0 0  ${waist_offset_z}" rpy="0 0 0"/>
+    <joint name="hip_joint" type="revolute">
+      <origin xyz="0 0  ${hip_offset_z}" rpy="0 0 0"/>
       <axis xyz="0 1 0"/>
-      <limit lower="${waist_llimit}" upper="${waist_ulimit}" velocity="${waist_vlimit}" effort="1.0" />
+      <limit lower="${hip_llimit}" upper="${hip_ulimit}" velocity="${hip_vlimit}" effort="1.0" />
       <parent link="femur_link"/>
       <child link="torso_link"/>

File: sheldon_description/urdf/sheldon.urdf (robot description, URDF)
Before this commit: robot sheldon_robot, 55 links, 54 joints
Joints:
- removed joint waist_joint
- added joint hip_joint: type revolute, parent femur_link, child torso_link, origin xyz=0 0  0.28 rpy=0 0 0, axis 0 1 0, limit lower=-0.175 upper=1.92 effort=1.0 velocity=1.571

Commit message: added chest camera

File: sheldon_description/urdf/body.urdf.xacro (robot description, xacro)
@@ -26,4 +26,11 @@
   <xacro:property name="torso_size_y" value="0.355" />
   <xacro:property name="torso_size_z" value="0.457" />  <!--  to top of shoulder .5112 .7112 28 inch torso for now -->
+   <xacro:property name="chest_camera_servo_offset_x" value="0.090" />
+   <xacro:property name="chest_camera_servo_offset_y" value="-0.098" />
+   <xacro:property name="chest_camera_servo_offset_z" value="0.380" /> <!-- 350 from bottom of torso? -->
+   <xacro:property name="chest_camera_offset_x" value="-0.044" />
+   <xacro:property name="chest_camera_offset_y" value="0.0" />
+   <xacro:property name="chest_camera_offset_z" value="0.08" />
+   <xacro:property name="chest_camera_rotation" value="0.0" />
   <xacro:macro name="body" params="parent name color">
     <!-- Base to lower leg link -->
@@ -94,4 +101,18 @@
       </collision>
     </link>
+    <!-- Chest Camera Servo -->
+      <origin xyz="0 0 0" rpy="0 0 3.14"/>
+    <dynamixel_rx28_pan parent="torso_link" name="chest_camera_servo" color="DarkGrey">
+    <origin xyz="${chest_camera_servo_offset_x} ${chest_camera_servo_offset_y} ${chest_camera_servo_offset_z}"
+            rpy="0 -1.57 -1.57" />
+    </dynamixel_rx28_pan>
+     <rx28_side_revolute parent="chest_camera_servo_link" name="chest_camera_tilt" llimit="-0.785" ulimit="0.785" vlimit="5.8" color="${servo_bracket_color}" >
+      <origin xyz="0 0 ${(rx28_servo_width/2)+0.003}" rpy="0 0 0"/>
+    </rx28_side_revolute>
+    <!-- Attach Astra camera  -->
+  <astra_camera name = "astra_camera" parent = "chest_camera_tilt" color="Green">
+     <origin xyz="${chest_camera_offset_x} ${chest_camera_offset_y} ${chest_camera_offset_z}"
+     rpy="1.57 0 1.57" />
+  </astra_camera>
   </xacro:macro>
 </robot>

File: sheldon_description/urdf/head.urdf.xacro (robot description, xacro)
@@ -8,5 +8,5 @@
    <xacro:property name="head_depth_camera_offset_x" value="0.050" />
    <xacro:property name="head_depth_camera_offset_y" value="0.000" />
-   <xacro:property name="head_depth_camera_offset_z" value="0.025" /> <!-- 350 from bottom of torso? -->
+   <xacro:property name="head_depth_camera_offset_z" value="0.080" /> <!-- 1.250m from ground -->
    <xacro:property name="head_depth_camera_tilt" value="0.16" /> <!-- rotation  -->
   <xacro:macro name="head" params="name parent color *origin">
@@ -34,5 +34,5 @@
     <!-- Side Tilt -->
     <dynamixel_rx28_tilt parent="${name}_tilt_link" name="${name}_sidetilt_servo" color="DarkGrey">
-      <origin xyz="${0.0611-0.013+0.0045 + (0.032/2)} 0 0" rpy="-1.57 0 0"/>
+      <origin xyz="${0.0611 + 0.0045 + (0.032/2)} 0 0" rpy="-1.57 0 0"/>
     </dynamixel_rx28_tilt>
     <rx28_hinge parent="${name}_sidetilt_servo_link" name="${name}_sidetilt" llimit="-0.35" ulimit="0.35" vlimit="0.524" color="Grey">

File: sheldon_description/urdf/robot.urdf.xacro (robot description, xacro)
@@ -53,8 +53,4 @@
    </depth_camera>
 -->
-   <!-- Attach Astra camera in the chest  -->
-  <astra_camera name = "astra_camera" parent = "torso" color="Green">
-     <origin xyz="${front_astra_camera_offset_x} ${front_astra_camera_offset_y} ${front_astra_camera_offset_z}" rpy="0 ${front_astra_camera_rotation} 0" />
-  </astra_camera>
 <!--
    <sensor_lplidar parent = "base">

Commit message: joint states service WIP

File: sheldon_description/urdf/body.urdf.xacro (robot description, xacro)
@@ -56,5 +56,5 @@
       </collision>
     </link>
-    <joint name="knee_joint" type="revolute">
+    <joint name="knee_bend_joint" type="revolute">
       <origin xyz="0 0  ${knee_offset_z}" rpy="0 0 0"/>
       <axis xyz="0 -1 0"/>
@@ -79,5 +79,5 @@
       </collision>
     </link>
-    <joint name="hip_joint" type="revolute">
+    <joint name="hip_bend_joint" type="revolute">
       <origin xyz="0 0  ${hip_offset_z}" rpy="0 0 0"/>
       <axis xyz="0 1 0"/>

File: sheldon_description/urdf/sheldon.urdf (robot description, URDF)
Before this commit: robot sheldon_robot, 55 links, 54 joints
Joints:
- removed joint hip_joint
- removed joint knee_joint
- added joint hip_bend_joint: type revolute, parent femur_link, child torso_link, origin xyz=0 0  0.281 rpy=0 0 0, axis 0 1 0, limit lower=-0.175 upper=1.92 effort=1.0 velocity=1.571
- added joint knee_bend_joint: type revolute, parent tibia_link, child femur_link, origin xyz=0 0  0.109 rpy=0 0 0, axis 0 -1 0, limit lower=-0.175 upper=0.873 effort=1.0 velocity=1.571
